Commit message: added arms to cob4-7

File: cob_hardware_config/robots/cob4-7/urdf/calibration_default.urdf.xacro (robot description, xacro)
@@ -49,4 +49,18 @@
 	<xacro:property name="def_sensorring_pitch" value="0.0"/>
 	<xacro:property name="def_sensorring_yaw" value="0.0"/>
+	<!-- arm right mount positions | relative to torso_3_link -->
+	<xacro:property name="def_arm_right_x" value="0.0"/>
+	<xacro:property name="def_arm_right_y" value="-0.014"/>
+	<xacro:property name="def_arm_right_z" value="0.55"/>
+	<xacro:property name="def_arm_right_roll" value="1.57097"/>
+	<xacro:property name="def_arm_right_pitch" value="0"/>
+	<xacro:property name="def_arm_right_yaw" value="0.0"/>
+	<!-- arm left mount positions | relative to torso_3_link -->
+	<xacro:property name="def_arm_left_x" value="0.0"/>
+	<xacro:property name="def_arm_left_y" value="0.014"/>
+	<xacro:property name="def_arm_left_z" value="0.55"/>
+	<xacro:property name="def_arm_left_roll" value="1.57097"/>
+	<xacro:property name="def_arm_left_pitch" value="0"/>
+	<xacro:property name="def_arm_left_yaw" value="3.14159"/>
 	<!-- *********************************** -->
 	<!-- kinematic chain reference positions -->

File: cob_hardware_config/robots/cob4-7/urdf/cob4-7.urdf.xacro (robot description, xacro)
@@ -11,4 +11,8 @@
   <!-- torso -->
   <xacro:include filename="$(find cob_description)/urdf/cob4_torso/torso.urdf.xacro" />
+  <!-- arm -->
+  <xacro:include filename="$(find cob_description)/urdf/cob4_arm/cob4_arm.urdf.xacro" />
+  <!-- hand -->
+  <xacro:include filename="$(find cob_description)/urdf/cob4_gripper/gripper.urdf.xacro" />
   <!-- head -->
   <xacro:include filename="$(find cob_description)/urdf/cob4_head/head.urdf.xacro" />
@@ -53,4 +57,10 @@
     <origin xyz="${head_cam_x} ${head_cam_y} ${head_cam_z}" rpy="${head_cam_roll} ${head_cam_pitch} ${head_cam_yaw}" />
   </xacro:usb_cam>
+  <xacro:cob4_arm name="arm_right" parent="torso_3_link" has_podest="false">
+    <origin xyz="${arm_right_x} ${arm_right_y} ${arm_right_z}" rpy="${arm_right_roll} ${arm_right_pitch} ${arm_right_yaw}" />
+  </xacro:cob4_arm>
+  <xacro:cob4_arm name="arm_left" parent="torso_3_link" has_podest="false">
+    <origin xyz="${arm_left_x} ${arm_left_y} ${arm_left_z}" rpy="${arm_left_roll} ${arm_left_pitch} ${arm_left_yaw}" />
+  </xacro:cob4_arm>
   <xacro:sensorring name="sensorring" parent="head_3_link" active="true">
     <origin xyz="${sensorring_x} ${sensorring_y} ${sensorring_z}" rpy="${sensorring_roll} ${sensorring_pitch} ${sensorring_yaw}" />

File: cob_hardware_config/robots/cob4-7/urdf/properties.urdf.xacro (robot description, xacro)
@@ -52,4 +52,18 @@
 	<xacro:property name="sensorring_pitch" value="${def_sensorring_pitch+offset_sensorring_pitch}"/>
 	<xacro:property name="sensorring_yaw" value="${def_sensorring_yaw+offset_sensorring_yaw}"/>
+	<!-- arm mount positions | relative to torso_3_link -->
+	<xacro:property name="arm_right_x" value="${def_arm_right_x+offset_arm_right_x}"/>
+	<xacro:property name="arm_right_y" value="${def_arm_right_y+offset_arm_right_y}"/>
+	<xacro:property name="arm_right_z" value="${def_arm_right_z+offset_arm_right_z}"/>
+	<xacro:property name="arm_right_roll" value="${def_arm_right_roll+offset_arm_right_roll}"/>
+	<xacro:property name="arm_right_pitch" value="${def_arm_right_pitch+offset_arm_right_pitch}"/>
+	<xacro:property name="arm_right_yaw" value="${def_arm_right_yaw+offset_arm_right_yaw}"/>
+	<!-- arm mount positions | relative to torso_3_link -->
+	<xacro:property name="arm_left_x" value="${def_arm_left_x+offset_arm_left_x}"/>
+	<xacro:property name="arm_left_y" value="${def_arm_left_y+offset_arm_left_y}"/>
+	<xacro:property name="arm_left_z" value="${def_arm_left_z+offset_arm_left_z}"/>
+	<xacro:property name="arm_left_roll" value="${def_arm_left_roll+offset_arm_left_roll}"/>
+	<xacro:property name="arm_left_pitch" value="${def_arm_left_pitch+offset_arm_left_pitch}"/>
+	<xacro:property name="arm_left_yaw" value="${def_arm_left_yaw+offset_arm_left_yaw}"/>
 	<!-- *********************************** -->
 	<!-- kinematic chain reference positions -->
